Commit message: add world link, update imu_link and joints

File: dare_code/robot_description/canary.xacro (robot description, xacro)
@@ -9,7 +9,14 @@
   </material>
   <!-- Base Properties -->
-  <xacro:property name="body_length" value="0.2" />
-  <xacro:property name="body_width" value="0.1" />
-  <xacro:property name="body_height" value="0.05" />
+  <xacro:property name="body_length" value="0.8" />
+  <xacro:property name="body_width" value="0.3" />
+  <xacro:property name="body_height" value="0.5" />
+  <link name="world">
+  </link>
+  <joint name="world_joint" type="fixed">
+      <origin xyz="0 0 0.5" rpy="0 0 0" />
+      <parent link="world" />
+      <child link="base_link" />
+  </joint>
   <!-- Base Link -->
   <link name="base_link">
@@ -21,17 +28,7 @@
       <material name="blue"/>
     </visual>
-    <!--<collision>
-      <origin xyz="0 0 0" rpy="0 0 0" />
-      <geometry>
-        <box size="0.4 0.04 0.04"/>
-      </geometry>
-    </collision>-->
-    <!--<inertial>
-       <mass value="0.3"/>
-       <inertia ixx="1.0" ixy="0.0" ixz="0.0" iyy="1.0" iyz="0.0" izz="1.0"/>
-     </inertial>-->
   </link>
   <!-- Front Left Wing Link -->
-  <link name="front_left_wing">
+  <!--<link name="front_left_wing">
     <visual>
       <origin xyz="0.16 0.13 0" rpy="0 0 0" />
@@ -45,7 +42,7 @@
     <child link="front_left_wing"/>
     <origin xyz="0.16 0.13 0"/>
-  </joint>
+  </joint>-->
   <!-- Front Right Wing Link -->
-  <link name="front_right_wing">
+  <!-- <link name="front_right_wing">
     <visual>
       <origin xyz="0.16 -0.13 0" rpy="0 0 0" />
@@ -59,7 +56,7 @@
     <child link="front_right_wing"/>
     <origin xyz="0.16 -0.13 0"/>
-  </joint>
+  </joint> -->
   <!-- Back Left Wing Link -->
-  <link name="back_left_wing">
+  <!-- <link name="back_left_wing">
     <visual>
       <origin xyz="-0.09 0.13 0" rpy="0 0 0" />
@@ -73,7 +70,7 @@
     <child link="back_left_wing"/>
     <origin xyz="-0.09 0.13 0"/>
-  </joint>
+  </joint> -->
   <!-- Back Right Wing Link -->
-  <link name="back_right_wing">
+  <!-- <link name="back_right_wing">
     <visual>
       <origin xyz="-0.09 -0.13 0" rpy="0 0 0" />
@@ -87,19 +84,19 @@
     <child link="back_right_wing"/>
     <origin xyz="-0.09 -0.13 0"/>
-  </joint>
+  </joint> -->
   <!-- IMU Link -->
-  <link name="imu">
+  <link name="imu_link">
   </link>
-  <joint name="base_to_imu" type="fixed">
+  <joint name="imu_joint" type="fixed">
     <parent link="base_link"/>
-    <child link="imu"/>
+    <child link="imu_link"/>
     <origin xyz="0 0 0"/>
   </joint>
   <!-- Lidar above on base_link-->
-  <link name="lidar">
+  <link name="lidar_link">
   </link>
-  <joint name="base_to_lidar" type="fixed">
+  <joint name="lidar_joint" type="fixed">
     <parent link="base_link"/>
-    <child link="lidar"/>
+    <child link="lidar_link"/>
     <origin xyz="0 0 0.06"/>
   </joint>

Commit message: Update canary.xacro

File: dare_code/robot_description/canary.xacro (robot description, xacro)
@@ -94,9 +94,9 @@
   </joint>
   <!-- Lidar above on base_link-->
-  <link name="lidar_link">
+  <link name="laser_frame">
   </link>
   <joint name="lidar_joint" type="fixed">
     <parent link="base_link"/>
-    <child link="lidar_link"/>
+    <child link="laser_frame"/>
     <origin xyz="0 0 0.06"/>
   </joint>
